File: arduino-level-shifter-shield.kicad_pcb (KiCad board)
At the start: 2 copper layers, 56 x 53 mm, 51 parts, among them J1 VCC1_EXT_OUT, J2 VCC2_EXT_OUT, J3 VCC3_EXT, J41 POWER, J42 DIGITAL_D8_D13_I2C, J43 ANALOG_IN, J44 ICSP 1/2, J45 ICSP 2/2, J46 DIGITAL_D0_D7, J51 GP 1/2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

Commit message: Rev: 2
Parts:
- added J47: VREG_IN, Custom:PinHeader_1x03, F.Cu at (14.6, -16.5)
- J44: value ICSP 1/2 -> ICSP_1/2
- J45: value ICSP 2/2 -> ICSP_2/2
- J51: value GP 1/2 -> GP_VCC3
- J52: value GP 2/2 -> GP
- J53: value DIGITAL_D8_D13_I2C -> DIGITAL_D8_D13_I2C_VCC2
- J54: value ICSP 1/2 -> ICSP_VCC3_1/2
- J55: value ICSP 2/2 -> ICSP_VCC3_2/2
- J56: value DIGITAL_D0_D7 -> DIGITAL_D0_D7_VCC1
- moved J44 5.08 mm to (51.0, -30.5)
- moved J45 5.08 mm to (53.5, -30.5)
- moved J54 5.08 mm to (45.9, -30.5)
- moved J55 5.08 mm to (48.5, -30.5)
- moved SW1 2.54 mm to (53.3, -35.4)
- moved C14 1.46 mm to (46.4, -42.7)
- moved C24 1.46 mm to (24.5, -42.7)
- moved C15 1.46 mm to (46.3, -38.9)
- moved C25 1.46 mm to (24.5, -38.9)
- moved C35 1.38 mm to (43.6, -16.3)
- moved C34 1.38 mm to (39.8, -16.3)
- moved J1 0.20 mm to (38.3, -33.0)
Connections:
- C11 pad 1: +5V -> /VREG_IN
- C15 pad 1: +5V -> /IOREF
- C21 pad 1: +5V -> /VREG_IN
- C25 pad 1: +5V -> /IOREF
- C31 pad 1: +5V -> /VREG_IN
- C35 pad 1: +5V -> /IOREF
- J41 pad 2: unconnected-(J41-Pad2) -> /IOREF
- J41 pad 8: unconnected-(J41-Pad8) -> /VIN
- J45 pad 1: +5V -> unconnected-(J45-Pad1)
- U11 pad 3: +5V -> /VREG_IN
- U12 pad 19: +5V -> /IOREF
- U21 pad 3: +5V -> /VREG_IN
- U22 pad 19: +5V -> /IOREF
- U31 pad 3: +5V -> /VREG_IN
- U32 pad 19: +5V -> /IOREF
Routing:
- net +5V: track 152.3 -> 23.1 mm, vias 5 -> 1
- net /IOREF: track 0.00 -> 94.3 mm, vias 0 -> 4
- net /VREG_IN: track 0.00 -> 38.5 mm, vias 0 -> 1
- net /VIN: track 0.00 -> 22.9 mm
- net /VCC3: track 79.3 -> 97.7 mm
- net /VCC1_REG: track 35.8 -> 46.2 mm, vias 0 -> 1
- net /VCC1_EXT: track 13.5 -> 20.6 mm
- net /VCC1: track 45.3 -> 38.4 mm
- net /MISO_A: track 15.0 -> 20.0 mm
- net /SCK_A: track 14.1 -> 19.1 mm
- net /RESET_A: track 12.7 -> 17.8 mm
- net /RESET_B: track 11.9 -> 16.7 mm
- net /MOSI_B: track 17.0 -> 21.2 mm
- net /SCK_B: track 14.3 -> 18.3 mm
- net /MOSI_A: track 18.5 -> 22.5 mm
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Other:
- board text added: "Arduino Logic Level Shifter Shield Rev: 2 www.petrvlasak.net"
- board text added: "VCC REG IN"
- board text removed: "Arduino Logic Level Shifter Shield Rev: 1 www.petrvlasak.net"
