File: arduino-level-shifter-shield.kicad_sch (KiCad schematic)
At the start: 51 parts, among them J1 VCC1_EXT_OUT, J2 VCC2_EXT_OUT, J3 VCC3_EXT, J41 POWER, J42 DIGITAL_D8_D13_I2C, J43 ANALOG_IN, J44 ICSP 1/2, J45 ICSP 2/2, J46 DIGITAL_D0_D7, J51 GP 1/2, J52 GP 2/2, J53 DIGITAL_D8_D13_I2C, J54 ICSP 1/2, J55 ICSP 2/2, J56 DIGITAL_D0_D7, SW1 VCC1_SELECT, SW2 VCC2_SELECT, SW3 VCC3_SELECT, U11 LM317_TO-252, U12 TXS0108EPWR, U21 LM317_TO-252, U22 TXS0108EPWR, U31 LM317_TO-252, U32 TXS0108EPWR

Commit message: Rev: 2
Parts:
- added J47: VREG_IN, Custom:PinHeader_1x03, symbol Connector_Generic:Conn_01x03
- J44: value ICSP 1/2 -> ICSP_1/2
- J45: value ICSP 2/2 -> ICSP_2/2
- J51: value GP 1/2 -> GP_VCC3
- J52: value GP 2/2 -> GP
- J53: value DIGITAL_D8_D13_I2C -> DIGITAL_D8_D13_I2C_VCC2
- J54: value ICSP 1/2 -> ICSP_VCC3_1/2
- J55: value ICSP 2/2 -> ICSP_VCC3_2/2
- J56: value DIGITAL_D0_D7 -> DIGITAL_D0_D7_VCC1
Connections:
- net +5V: now also J47.1 (Pin_1); no longer C11.1, C15.1, C21.1, C25.1, C31.1, C35.1, J45.1 (Pin_1), U11.3 (VI), U12.19 (VCCB), U21.3 (VI), U22.19 (VCCB), U31.3 (VI), U32.19 (VCCB)
- net IOREF: now reaches J41.2 (Pin_2)
- net IOREF: now also C15.1, C25.1, C35.1, U12.19 (VCCB), U22.19 (VCCB), U32.19 (VCCB)
- net VIN: now reaches J41.8 (Pin_8)
- net VIN: now also J47.3 (Pin_3)
- new net VREG_IN: C11.1, C21.1, C31.1, J47.2 (Pin_2), U11.3 (VI), U21.3 (VI), U31.3 (VI)
- no-connect marks 12 -> 11
Other:
- moved on the sheet: J44, J45
